File: KiCAD/Helios-Display.kicad_sch (KiCad schematic)
At the start: 3 parts, among them J1 Raspberry_Pi_2_3, J2 FFC_ST1633 (Touch), J3 Conn_01x45_Female

Commit message: updated KiCAD files
Parts:
- added C1: 470nF, Capacitor_SMD:C_0603_1608Metric_Pad1.08x0.95mm_HandSolder, symbol Device:C
- added C2: 4.7uF/16V, Capacitor_SMD:C_1210_3225Metric_Pad1.33x2.70mm_HandSolder, symbol Device:C
- added C3: 220uF/16V, Capacitor_SMD:CP_Elec_6.3x3, symbol Device:C_Polarized
- added C4: 0.47uF, Capacitor_SMD:C_0805_2012Metric_Pad1.18x1.45mm_HandSolder, symbol Device:C
- added C5: 100nF, Capacitor_SMD:C_0603_1608Metric_Pad1.08x0.95mm_HandSolder, symbol Device:C
- added C6: NC, Capacitor_SMD:C_0603_1608Metric_Pad1.08x0.95mm_HandSolder, symbol Device:C
- added C7: 4.7uF/25V, Capacitor_SMD:C_1210_3225Metric_Pad1.33x2.70mm_HandSolder, symbol Device:C
- added C8: 22uF/25V, Capacitor_SMD:CP_Elec_6.3x3, symbol Device:C_Polarized
- added D1: B360, Diode_SMD:D_SMC, symbol Diode:B360
- added F1: Fuse, Fuse:Fuse_1206_3216Metric_Pad1.42x1.75mm_HandSolder, symbol Device:Fuse
- added H1, H2, H3, H4: MountingHole_Pad, MountingHole:MountingHole_3mm_Pad_Via, symbol Mechanical:MountingHole_Pad
- added H5, H6, H7, H8: MountingHoleRaspi, MountingHole:MountingHole_2.5mm, symbol Mechanical:MountingHole
- added J4: Power, Connector_PinHeader_2.54mm:PinHeader_1x03_P2.54mm_Vertical, symbol Connector_Generic:Conn_01x03
- added J5: LED_BL, Connector_PinHeader_2.54mm:PinHeader_1x04_P2.54mm_Vertical, symbol Connector_Generic:Conn_01x04
- added J6: I2C, Connector_PinHeader_2.54mm:PinHeader_1x04_P2.54mm_Vertical, symbol Connector_Generic:Conn_01x04
- added J7: GPIO, Connector_PinHeader_2.54mm:PinHeader_1x03_P2.54mm_Vertical, symbol Connector_Generic:Conn_01x03
- added J8: Raspberry_Pi_2_3, Connector_PinHeader_2.54mm:PinHeader_2x20_P2.54mm_Vertical_SMD, symbol Connector:Raspberry_Pi_2_3
- added L1: 33uH/3.5A, Inductor_SMD:L_12x12mm_H8mm, symbol Device:L
- added M1: AM4490N, Package_SO:SOIC-8_3.9x4.9mm_P1.27mm, symbol Helios-Display:AM4490N
- added R1: 270, Resistor_SMD:R_0603_1608Metric_Pad0.98x0.95mm_HandSolder, symbol Device:R
- added R10, R13, R14, R7, R9: 0, Resistor_SMD:R_0603_1608Metric_Pad0.98x0.95mm_HandSolder, symbol Device:R
- added R11, R12: 50, Resistor_SMD:R_0603_1608Metric_Pad0.98x0.95mm_HandSolder, symbol Device:R
- added R2, R4: 100k, Resistor_SMD:R_0603_1608Metric_Pad0.98x0.95mm_HandSolder, symbol Device:R
- added R3: R, Resistor_SMD:R_0603_1608Metric_Pad0.98x0.95mm_HandSolder, symbol Device:R
- added R5: 10, Resistor_SMD:R_0603_1608Metric_Pad0.98x0.95mm_HandSolder, symbol Device:R
- added R6: 50m, Resistor_SMD:R_1206_3216Metric_Pad1.30x1.75mm_HandSolder, symbol Device:R
- added R8: NC, Resistor_SMD:R_1206_3216Metric_Pad1.30x1.75mm_HandSolder, symbol Device:R
- added U1: MP3385A, Package_DFN_QFN:QFN-20-1EP_4x4mm_P0.5mm_EP2.5x2.5mm_ThermalVias, symbol Helios-Display:MP3385A
- J1: footprint Connector_PinHeader_2.54mm:PinHeader_2x20_P2.54mm_Vertical -> Connector_PinHeader_2.54mm:PinHeader_2x20_P2.54mm_Vertical_SMD
- J3: value Conn_01x45_Female -> FFC_LCD; footprint (none) -> Connector_FFC-FPC:Hirose_FH12-45S-0.5SH_1x45-1MP_P0.50mm_Horizontal
Connections:
- net LCD_B_{0} is gone; now on net GNDA: J3.21 (Pin_21)
- net LCD_B_{1} is gone; now on net GNDA: J3.22 (Pin_22)
- net LCD_DISP is gone; now on net +3V3: J3.31 (Pin_31)
- net LCD_G_{0} is gone; now on net GNDA: J3.13 (Pin_13)
- net LCD_G_{1} is gone; now on net GNDA: J3.14 (Pin_14)
- net LCD_LED_A2 is gone; now on net LCD_LED_A1: J3.45 (Pin_45)
- net LCD_R_{0} is gone; now on net GNDA: J3.5 (Pin_5)
- net LCD_R_{1} is gone; now on net GNDA: J3.6 (Pin_6)
- net +3V3: now also J2.3 (Pin_3), J4.3 (Pin_3), J6.4 (Pin_4), J8.1 (3V3), J8.17 (3V3), R11.2, R12.2, U1.3 (EN); no longer J2.4 (Pin_4)
- net +5V: now also F1.1, J4.2 (Pin_2), J8.2 (5V), J8.4 (5V)
- net GPIO_SCL: now also J2.4 (Pin_4), J6.3 (Pin_3), J8.18 (GPIO24), R12.1, U1.6 (SCL); no longer J2.3 (Pin_3)
- net GPIO_SDA: now also J2.5 (Pin_5), J6.2 (Pin_2), J8.16 (GPIO23), R11.1, U1.7 (SDA); no longer J2.2 (Pin_2)
- net LCD_B_{2}: now also J8.7 (GCLK0/GPIO4)
- net LCD_B_{3}: now also J8.29 (GCLK1/GPIO5)
- net LCD_B_{4}: now also J8.31 (GCLK2/GPIO6)
- net LCD_B_{5}: now also J8.26 (~{CE1}/GPIO7)
- net LCD_B_{6}: now also J8.24 (~{CE0}/GPIO8)
- net LCD_B_{7}: now also J8.21 (MISO0/GPIO9)
- net LCD_DE: now also J8.28 (ID_SC/GPIO1)
- net LCD_G_{2}: now also J8.19 (MOSI0/GPIO10)
- net LCD_G_{3}: now also J8.23 (SCLK0/GPIO11)
- net LCD_G_{4}: now also J8.32 (PWM0/GPIO12)
- net LCD_G_{5}: now also J8.33 (PWM1/GPIO13)
- net LCD_G_{6}: now also J8.8 (GPIO14/TXD)
- net LCD_G_{7}: now also J8.10 (GPIO15/RXD)
- net LCD_HSYNC: now also J8.5 (SCL/GPIO3)
- net LCD_LED_A1: now also C7.1, C8.1, D1.1 (K), J5.2 (Pin_2), J5.4 (Pin_4), R9.2
- net LCD_LED_C1: now also J5.1 (Pin_1), R14.2
- net LCD_LED_C2: now also J5.3 (Pin_3), R13.2
- net LCD_PCLK: now also J8.27 (ID_SD/GPIO0)
- net LCD_R_{2}: now also J8.36 (GPIO16)
- net LCD_R_{3}: now also J8.11 (GPIO17)
- net LCD_R_{4}: now also J8.12 (GPIO18/PWM0)
- net LCD_R_{5}: now also J8.35 (GPIO19/MISO1)
- net LCD_R_{6}: now also J8.38 (GPIO20/MOSI1)
- net LCD_R_{7}: now also J8.40 (GPIO21/SCLK1)
- net LCD_VSYNC: now also J8.3 (SDA/GPIO2)
- net ST1633_IRQ: now also J2.2 (Pin_2), J8.15 (GPIO22); no longer J2.5 (Pin_5)
- net GPIO27: now reaches J1.13 (GPIO27)
- net GPIO27: now also J7.3 (Pin_3), J8.13 (GPIO27)
- net GPIO25: now reaches J1.22 (GPIO25)
- net GPIO25: now also J7.1 (Pin_1), J8.22 (GPIO25)
- net GPIO26: now reaches J1.37 (GPIO26)
- net GPIO26: now also J7.2 (Pin_2), J8.37 (GPIO26)
- net GNDA: now reaches J2.6 (Pin_6)
- net GNDA: now also J1.14 (GND), J1.20 (GND), J1.25 (GND), J1.30 (GND), J1.34 (GND), J1.39 (GND), J1.6 (GND), J1.9 (GND), J3.1 (Pin_1), J3.2 (Pin_2), J3.29 (Pin_29), J3.40 (Pin_40), J3.41 (Pin_41), C1.2, C2.2, C3.2, C4.1, C5.2, C6.2, C7.2, C8.2, H1.1, H2.1, H3.1, H4.1, J4.1 (Pin_1), J6.1 (Pin_1), J8.14 (GND), J8.20 (GND), J8.25 (GND), J8.30 (GND), J8.34 (GND), J8.39 (GND), J8.6 (GND), J8.9 (GND), R2.1, R3.2, R6.2, U1.21 (GND)
- removed net GNDPWR: J1.14 (GND), J1.20 (GND), J1.25 (GND), J1.30 (GND), J1.34 (GND), J1.39 (GND), J1.6 (GND), J1.9 (GND), J2.1 (Pin_1), J3.1 (Pin_1), J3.2 (Pin_2), J3.29 (Pin_29), J3.40 (Pin_40), J3.41 (Pin_41)
- new net: R14.1, U1.16 (LED2)
- new net: R9.1, U1.18 (OVP)
- new net: R4.2, U1.8 (FT)
- new net: C2.1, C3.1, F1.2, L1.1, R7.1
- new net: D1.2 (A), L1.2, M1.1 (D)
- new net: C6.1, R10.1, U1.19 (IS)
- new net: M1.5 (S), R10.2, R6.1, R8.2
- new net: M1.4 (G), R5.2
- new net: R5.1, U1.1 (DRV)
- new net: C5.1, U1.9 (LPF)
- new net: R2.2, U1.10 (OSC)
- new net: C1.1, R1.2
- new net: R3.1, U1.12 (ISET)
- new net: R13.1, U1.17 (LED1)
- new net: R1.1, U1.11 (COMP)
- new net: R8.1, U1.15 (PGND)
- new net: R7.2, U1.4 (VIN)
- new net GND: U1.20 (AGND)
- new net VCC: C4.2, R4.1, U1.2 (VCC)
- no-connect marks 8 -> 9
Other:
- company: (none) -> morlac.de
- title: (none) -> Helios-Display Adapter (RPi)
- moved on the sheet: J1, J2, J3
